File: KiCad - Main/steering.kicad_pcb (KiCad board)
At the start: 2 copper layers, 67 x 33 mm, 40 parts, among them J1 USB_C_Receptacle_USB2.0_14P, J2 Conn_01x04_Pin, J3 Conn_01x06_Socket, J4 Conn_01x03_Socket A1324LLHLT-T, J5 Conn_01x03_Socket A1324LLHLT-T, J6 Conn_01x02_Socket USART2, SW1 SW_Push, SW2 SW_SPDT, U1 STM32F732RET6, U2 USBLC6-2SC6, U3 AP2112K-3.3, Y1 16MHz

Commit message: BOM, pcbway stuff, and final check over
Parts:
- C11, C12: value 12pF -> 10pF
- C7: footprint Capacitor_SMD:C_0805_2012Metric_Pad1.18x1.45mm_HandSolder -> Capacitor_SMD:C_0603_1608Metric_Pad1.08x0.95mm_HandSolder
