File: KiCad - Main/steering.kicad_sch (KiCad schematic)
At the start: 36 parts, among them J1 USB_C_Receptacle_USB2.0_14P, J2 Conn_01x04_Pin, J3 Conn_01x06_Socket, J4 Conn_01x03_Socket A1324LLHLT-T, J5 Conn_01x03_Socket A1324LLHLT-T, J6 Conn_01x02_Socket USART2, SW1 SW_Push, SW2 SW_SPDT, U1 STM32F732RET6, U2 USBLC6-2SC6, U3 AP2112K-3.3, Y1 16MHz

Commit message: BOM, pcbway stuff, and final check over
Parts:
- added J7: Conn_01x21_Socket, Connector_PinHeader_2.54mm:PinHeader_1x21_P2.54mm_Vertical, symbol Connector:Conn_01x21_Socket
- added J8: Conn_01x15_Socket, Connector_PinHeader_2.54mm:PinHeader_1x15_P2.54mm_Vertical, symbol Connector:Conn_01x15_Socket
- C1, C10, C2, C3, C4, C5: Link (none) -> https://www.digikey.com/en/products/detail/murata-electroni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; MF (none) -> Murata Electronics; MP (none) -> GCM188L81H104KA57D; Price (none) -> $0.14
- C11, C12: value 12pF -> 10pF; Link (none) -> https://www.digikey.com/en/products/detail/murata-electroni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; MF (none) -> Murata Electronics; MP (none) -> GCM1555C1H100JA16D; Price (none) -> $0.11
- C14, C15, C8, C9: Link (none) -> https://www.digikey.com/en/products/detail/murata-electroni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; MF (none) -> Murata Electronics; MP (none) -> GRT188C8YA105KE13D; Price (none) -> $0.17
- C16: Link (none) -> https://www.digikey.com/en/products/detail/murata-electroni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; MF (none) -> Murata Electronics; MP (none) -> GRT188R61H225KE13D; Price (none) -> $0.2
- C17, C6: Link (none) -> https://www.digikey.ca/en/products/detail/murata-electronic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; MF (none) -> Murata Electronics; MP (none) -> GCJ21BR71A106KE01L; Price (none) -> $0.74
- C7: footprint Capacitor_SMD:C_0805_2012Metric_Pad1.18x1.45mm_HandSolder -> Capacitor_SMD:C_0603_1608Metric_Pad1.08x0.95mm_HandSolder; Link (none) -> https://www.digikey.ca/en/products/detail/murata-electronic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; MF (none) -> Murata Electronics; MP (none) -> GCM188R72A103KA37D; Price (none) -> $0.15
- D1: Link (none) -> https://www.digikey.com/en/products/detail/w%C3%BCrth-elekt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; MF (none) -> Wurth Elektronik; MP (none) -> 150060RS75000; Price (none) -> $0.15
- D2: Link (none) -> https://www.digikey.ca/en/products/detail/kyocera-avx/GG060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; MF (none) -> KYOCERA AVX; MP (none) -> GG060305100N2P; Price (none) -> $0.45
- F1: Link (none) -> https://www.digikey.ca/en/products/detail/yageo/SMD0603B050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; MF (none) -> YAGEO; MP (none) -> SMD0603B050TF; Price (none) -> $0.36
- FB1: Link (none) -> https://www.digikey.ca/en/products/detail/murata-electronic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; MF (none) -> Murata Electronics; MP (none) -> BLM18AG121SN1D; Price (none) -> $0.16
- J1: Link (none) -> https://www.digikey.com/en/products/detail/gct/USB4085-GF-A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; MF (none) -> GCT; MP (none) -> USB4085-GF-A; Price (none) -> $0.91
- R1: Link (none) -> https://www.digikey.com/en/products/detail/panasonic-indust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; MF (none) -> Panasonic Industry; MP (none) -> ERJ-3EKF1002V; Price (none) -> $0.1
- R2, R3: Link (none) -> https://www.digikey.com/en/products/detail/panasonic-indust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; MF (none) -> Panasonic Industry; MP (none) -> ERJ-3EKF5101V; Price (none) -> $0.15
- R4: Link (none) -> https://www.digikey.ca/en/products/detail/panasonic-industr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; MF (none) -> Panasonic Industry; MP (none) -> ERJ-PA3F1000V; Price (none) -> $0.24
- SW1: Link (none) -> https://www.digikey.com/en/products/detail/alps-alpine/SKSG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; MF (none) -> Alps Alpine; MP (none) -> SKSGACE010; Price (none) -> $0.45
- SW2: Link (none) -> https://www.digikey.com/en/products/detail/w%C3%BCrth-elekt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; Price (none) -> $2.51
- U1: Link (none) -> https://www.digikey.com/en/products/detail/stmicroelectroni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; MF (none) -> STMicroelectronics; MP (none) -> STM32F732RET6; Price (none) -> $15.43
- U2: Link (none) -> https://www.digikey.com/en/products/detail/shenzhen-slkormi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; MF (none) -> Shenzhen Slkormicro Semicon Co., Ltd.; MP (none) -> USBLC6-2SC6; Price (none) -> $0.18
- U3: Link (none) -> https://www.digikey.com/en/products/detail/diodes-incorpora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; MF (none) -> Diodes Incorporated; MP (none) -> AP2112K-3.3TRG1; Price (none) -> $0.28
- Y1: Link (none) -> https://www.digikey.com/en/products/detail/jauch-quartz/Q-1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; MF (none) -> Jauch Quartz; MP (none) -> Q 16,0-JXS32-8-10/10-WA-LF; Price (none) -> $0.61
